File: esp_to_rs3232.kicad_pcb (KiCad board)
At the start: 2 copper layers, 35.6 x 31.5 mm, 21 parts, among them J1 USB_B_Micro, J2 Conn_01x04, J3 DB9_Female_MountingHoles, U1 AMS1117-3.3, U2 ESP-12F, U3 MAX3232

Commit message: update footprint
Signed-off-by: SchumyHao <schumyhaojl@126.com>
Parts:
- removed FLASH: SW_Push, Button_Switch_SMD:SW_SPST_B3U-1000P
- added SW1: SW_Push, Button_Switch_SMD:SW_SPST_PTS810, F.Cu at (188.6, 88.3)
- C1, C2: footprint Capacitor_Tantalum_SMD:CP_EIA-1608-08_AVX-J_Pad1.25x1.05mm_HandSolder -> Capacitor_Tantalum_SMD:CP_EIA-3216-18_Kemet-A_Pad1.58x1.35mm_HandSolder
- J1: footprint Connector_USB:USB_Micro-B_GCT_USB3076-30-A -> Connector_USB:USB_Micro-B_Molex_47346-0001
- J2: footprint Connector_PinHeader_1.27mm:PinHeader_1x04_P1.27mm_Vertical -> Connector_PinHeader_2.54mm:PinHeader_1x04_P2.54mm_Vertical
- moved TP1 1.14 mm to (194.3, 98.6)
- moved TP3 0.64 mm to (194.3, 94.6)
- moved TP2 0.51 mm to (194.3, 83.6)
- moved J2 0.38 mm to (194.3, 108.8)
Connections:
- J3 pad 1: Net-(J3-Pad1) -> (no net)
- J3 pad 4: Net-(J3-Pad4) -> (no net)
- J3 pad 6: Net-(J3-Pad6) -> (no net)
- J3 pad 7: Net-(J3-Pad7) -> (no net)
- J3 pad 8: Net-(J3-Pad8) -> (no net)
- J3 pad 9: Net-(J3-Pad9) -> (no net)
- U2 pad 1: Net-(U2-Pad1) -> (no net)
- U2 pad 11: Net-(U2-Pad11) -> (no net)
- U2 pad 17: Net-(U2-Pad17) -> (no net)
- U2 pad 18: Net-(U2-Pad18) -> (no net)
- U2 pad 19: Net-(U2-Pad19) -> (no net)
- U2 pad 2: Net-(U2-Pad2) -> (no net)
- U2 pad 20: Net-(U2-Pad20) -> (no net)
- U2 pad 21: Net-(U2-Pad21) -> (no net)
- U2 pad 22: Net-(U2-Pad22) -> (no net)
- U2 pad 6: Net-(U2-Pad6) -> (no net)
- U2 pad 7: Net-(U2-Pad7) -> (no net)
- U3 pad 10: Net-(U3-Pad10) -> (no net)
- U3 pad 7: Net-(U3-Pad7) -> (no net)
- U3 pad 8: Net-(U3-Pad8) -> (no net)
- U3 pad 9: Net-(U3-Pad9) -> (no net)
Routing:
- net Net-(R3-Pad2): track 18.3 -> 21.7 mm
- net Net-(J3-Pad2): track 23.0 -> 26.2 mm
- net +3V3: track 60.0 -> 62.6 mm
- net Net-(C1-Pad1): track 13.1 -> 11.3 mm
- net Net-(J2-Pad2): track 35.3 -> 36.3 mm
- net Net-(J3-Pad3): track 16.5 -> 15.7 mm
- net GND: track 15.1 -> 15.3 mm, vias 21 -> 15
- net /RXOUT: vias 1 -> 0
