File: esp_to_rs3232.sch (KiCad schematic (older format))
At the start: 21 parts, among them J1 USB_B_Micro, J2 Conn_01x04, J3 DB9_Female_MountingHoles, SW1 SW_Push, U1 AMS1117-3.3, U2 ESP-12F, U3 MAX3232

Commit message: update footprint
Signed-off-by: SchumyHao <schumyhaojl@126.com>
Parts:
- C1, C2: footprint Capacitor_Tantalum_SMD:CP_EIA-1608-08_AVX-J_Pad1.25x1.05mm_HandSolder -> Capacitor_Tantalum_SMD:CP_EIA-3216-18_Kemet-A_Pad1.58x1.35mm_HandSolder
- J1: footprint Connector_USB:USB_Micro-B_GCT_USB3076-30-A -> Connector_USB:USB_Micro-B_Molex_47346-0001
- J2: footprint Connector_PinHeader_1.27mm:PinHeader_1x04_P1.27mm_Vertical -> Connector_PinHeader_2.54mm:PinHeader_1x04_P2.54mm_Vertical
- SW1: footprint Button_Switch_SMD:SW_SPST_B3U-1000P -> Button_Switch_SMD:SW_SPST_PTS810
Changed lines of the file:
@@
 EESchema Schematic File Version 4
+LIBS:esp_to_rs3232-cache
 EELAYER 30 0
 EELAYER END
@@
 F 0 "J1" H 1207 1717 50  0000 C CNN
 F 1 "USB_B_Micro" H 1207 1626 50  0000 C CNN
-F 2 "Connector_USB:USB_Micro-B_GCT_USB3076-30-A" H 1300 1200 50  0001 C CNN
+F 2 "Connector_USB:USB_Micro-B_Molex_47346-0001" H 1300 1200 50  0001 C CNN
 F 3 "~" H 1300 1200 50  0001 C CNN
 	1    1150 1250
@@
 F 0 "C2" H 2815 1346 50  0000 L CNN
 F 1 "10uF" H 2815 1255 50  0000 L CNN
-F 2 "Capacitor_Tantalum_SMD:CP_EIA-1608-08_AVX-J_Pad1.25x1.05mm_HandSolder" H 2700 1300 50  0001 C CNN
+F 2 "Capacitor_Tantalum_SMD:CP_EIA-3216-18_Kemet-A_Pad1.58x1.35mm_HandSolder" H 2700 1300 50  0001 C CNN
 F 3 "~" H 2700 1300 50  0001 C CNN
 	1    2700 1300
@@
 F 0 "J2" H 6280 2796 50  0000 L CNN
 F 1 "Conn_01x04" H 6280 2751 50  0001 L CNN
-F 2 "Connector_PinHeader_1.27mm:PinHeader_1x04_P1.27mm_Vertical" H 6200 2850 50  0001 C CNN
+F 2 "Connector_PinHeader_2.54mm:PinHeader_1x04_P2.54mm_Vertical" H 6200 2850 50  0001 C CNN
 F 3 "~" H 6200 2850 50  0001 C CNN
 	1    6200 2850
@@
 F 0 "C1" H 1815 1346 50  0000 L CNN
 F 1 "10uF" H 1815 1255 50  0000 L CNN
-F 2 "Capacitor_Tantalum_SMD:CP_EIA-1608-08_AVX-J_Pad1.25x1.05mm_HandSolder" H 1700 1300 50  0001 C CNN
+F 2 "Capacitor_Tantalum_SMD:CP_EIA-3216-18_Kemet-A_Pad1.58x1.35mm_HandSolder" H 1700 1300 50  0001 C CNN
 F 3 "~" H 1700 1300 50  0001 C CNN
 	1    1700 1300
@@
 F 0 "SW1" V 5796 3552 50  0000 R CNN
 F 1 "SW_Push" V 5705 3552 50  0000 R CNN
-F 2 "Button_Switch_SMD:SW_SPST_B3U-1000P" H 5750 3800 50  0001 C CNN
+F 2 "Button_Switch_SMD:SW_SPST_PTS810" H 5750 3800 50  0001 C CNN
 F 3 "~" H 5750 3800 50  0001 C CNN
 	1    5750 3600

Commit message: change c2 value
Signed-off-by: SchumyHao <schumyhaojl@126.com>
Parts:
- C4: value NC -> 0.1uF
Changed lines of the file:
@@
 P 8750 2000
 F 0 "C4" H 8928 2046 50  0000 L CNN
-F 1 "NC" H 8928 1955 50  0000 L CNN
+F 1 "0.1uF" H 8928 1955 50  0000 L CNN
 F 2 "Capacitor_SMD:C_0603_1608Metric" H 8750 2000 50  0001 C CNN
 F 3 "~" H 8750 2000 50  0001 C CNN
